File: KosmoPulseMain/KosmoPulseMain.kicad_sch (KiCad schematic)
At the start: 47 parts, among them J1 OUT6, J10 OUT12, J11 OUT24, J2 OUT4, J3 OUT2, J4 OUT1, J5 OUT3, J6 OUT7, J7 OUT5, J8 1247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

Commit message: Added GND to BIT 6
Parts:
- C1: footprint ao_tht:C_Disc_D3.0mm_W1.6mm_P2.50mm -> ao_tht:C_Rect_L7.2mm_W2.5mm_P5.00mm_FKS2_FKP2_MKS2_MKP2
Connections:
- net GND: now also J1.S, R12.2
Changed lines of the file:
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@@
   (junction (at 146.05 43.18) (diameter 0) (color 0 0 0 0)
+  )
+  (junction (at 81.28 148.59) (diameter 0) (color 0 0 0 0)
   )
   (junction (at 82.55 106.68) (diameter 0) (color 0 0 0 0)
@@
     (property "Reference" "C1" (id 0) (at 218.44 115.57 90))
     (property "Value" "100n" (id 1) (at 218.44 118.11 90))
-    (property "Footprint" "ao_tht:C_Disc_D3.0mm_W1.6mm_P2.50mm" (id 2) (at 222.25 122.2248 0)
+    (property "Footprint" "ao_tht:C_Rect_L7.2mm_W2.5mm_P5.00mm_FKS2_FKP2_MKS2_MKP2" (id 2) (at 222.25 122.2248 0)
       (effects (font (size 1.27 1.27)) hide)
     )
@@
     (pin "T")
   )
+  (symbol (lib_id "power:GND") (at 81.28 148.59 0) (unit 1)
+    (in_bom yes) (on_board yes) (fields_autoplaced)
+    (property "Reference" "#PWR?" (id 0) (at 81.28 154.94 0)
+      (effects (font (size 1.27 1.27)) hide)
+    )
+    (property "Value" "GND" (id 1) (at 81.28 153.67 0))
+    (property "Footprint" "" (id 2) (at 81.28 148.59 0)
+      (effects (font (size 1.27 1.27)) hide)
+    )
+    (property "Datasheet" "" (id 3) (at 81.28 148.59 0)
+      (effects (font (size 1.27 1.27)) hide)
+    )
+    (pin "1")
+  )
   (symbol (lib_id "ao_symbols:R") (at 74.93 124.46 90) (unit 1)
     (in_bom yes) (on_board yes)
@@
       (reference "#PWR012") (unit 1) (value "GND") (footprint "")
     )
+    (path "/e209ad97-34aa-4a0a-9cdc-ff05f470017b"
+      (reference "#PWR?") (unit 1) (value "GND") (footprint "")
+    )
     (path "/4e8cbbf0-a19f-49cc-8324-0b2e960fad6a"
-      (reference "C1") (unit 1) (value "100n") (footprint "ao_tht:C_Disc_D3.0mm_W1.6mm_P2.50mm")
+      (reference "C1") (unit 1) (value "100n") (footprint "ao_tht:C_Rect_L7.2mm_W2.5mm_P5.00mm_FKS2_FKP2_MKS2_MKP2")
     )
     (path "/13aad5e6-4db7-4272-9917-460d43d5f094"
